File: Igloo34/igloo34/igloo34.kicad_pcb (KiCad board)
At the start: 4 copper layers, 82 x 100 mm, 56 parts, among them J1 Conn_01x08_Pin, J10 Conn_01x10, J11 LSHM-120-02.5-L-DV-A-S-TR, J12 LSHM-120-02.5-L-DV-A-S-TR, J13 Conn_01x10, J14 Conn_01x10, J15 LSHM-120-02.5-L-DV-A-S-TR, J16 Conn_01x02, J17 Conn_01x02, J18 Conn_01x02, J19 Conn_01x02, J2 Conn_01x08_Pin, J20 LSHM-120-02.5-L-DV-A-S-TR, J21 Conn_01x02, J22 Conn_01x02, J23 Conn_01x02, J24 Conn_01x02, J3 BE40A-S-92SP-2-2-08-0152, J4 BE40A-S-92SP-2-2-08-0152, J5 Conn_01x08_Pin, J6 Conn_01x08_Pin, J7 LSHM-120-02.5-L-DV-A-S-TR, J8 LSHM-120-02.5-L-DV-A-S-TR, J9 Conn_01x10

Commit message: update
Parts:
- TP1, TP10, TP11, TP12, TP13, TP14, TP15, TP16, TP17, TP18, TP19, TP2, TP20, TP21, TP22, TP23, TP24, TP25, TP26, TP27, TP28, TP29, TP3, TP30, TP31, TP32, TP4, TP5, TP6, TP7, TP8, TP9: footprint TestPoint:TestPoint_THTPad_D1.0mm_Drill0.5mm -> 0_Library:Test point top pad
Routing:
- net GND: track 0.00 -> 19.0 mm, vias 0 -> 41
- net Net-(J9-Pin_3): track 44.9 -> 47.1 mm
- net Net-(J9-Pin_2): track 47.3 -> 49.5 mm
- net Net-(J9-Pin_4): track 43.5 -> 45.6 mm
- net Net-(J9-Pin_5): track 41.0 -> 43.0 mm
- net Net-(J9-Pin_1): track 48.6 -> 50.4 mm
- net Net-(J10-Pin_4): track 43.4 -> 45.1 mm
- net Net-(J9-Pin_6): track 39.6 -> 41.3 mm
- net Net-(J10-Pin_5): track 41.2 -> 42.9 mm
- net Net-(J10-Pin_1): track 49.1 -> 50.6 mm
- net Net-(J9-Pin_7): track 37.2 -> 38.7 mm
- net Net-(J10-Pin_2): track 47.4 -> 48.8 mm
- net Net-(J10-Pin_6): track 39.6 -> 41.0 mm
- net Net-(J10-Pin_3): track 45.1 -> 46.5 mm
- net Net-(J9-Pin_8): track 35.7 -> 37.1 mm
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Other:
- outline, holes or cut-outs redrawn
- board text added: "1"
- board text added: "10"
- board text added: "2"
- board text added: "3"
- board text added: "4"
- board text added: "5"
- board text added: "6"
- board text added: "7"
- board text added: "8"
- board text added: "9"
- board text added: "N"
- board text added: "Ryan Morgenstern Igloo34 Aug 2024"
- board text added: "S"
- board text added: "TODO:"
- board text removed: "Ryan Morgenstern Igloo30 Oct 2023"
- board text removed: "TODO: - A few via fence vias - Test points - Mounting holes - HUGE {dblquote}N{dblquote} and {dblquote}S{dblquote} (north/south) outside the dark box"
